Commit message: ft[structure]: Moves generic fabrics node to src so it can be derived.

File: fabrics_bridge/config/boxer.urdf (robot description, URDF)
Before this commit: robot albert, 7 links, 6 joints
Links:
- removed link base_link_ori
- removed link odom
- removed link world
- removed link world_base_link_x
- removed link world_base_link_y
- added link chassis_link, mass 250; collision mesh filename=meshes/collision/chassis_link.STL; visual mesh filename=meshes/visual/chassis_link.dae
- added link rotacastor_left_link, mass 1; collision cylinder length=0.001 radius=0.0625; visual cylinder length=0.06 radius=0.0625
- added link rotacastor_right_link, mass 1; collision cylinder length=0.001 radius=0.0625; visual cylinder length=0.06 radius=0.0625
- added link wheel_left_link, mass 10; collision cylinder length=0.001 radius=0.080; visual cylinder length=0.05 radius=0.080
- added link wheel_right_link, mass 10; collision cylinder length=0.001 radius=0.080; visual cylinder length=0.05 radius=0.080
- link base_link: mass None -> 1
- link ee_link: geometry visual sphere radius=0.0625
Joints:
- removed joint base_add_orientation
- removed joint boxer_joint_world
- removed joint world_base_theta
- removed joint world_base_x
- removed joint world_base_y
- added joint base_chassis_joint: type fixed, parent base_link, child chassis_link, origin xyz=0 0 0 rpy=0 0 0
- added joint rotacastor_left_joint: type continuous, parent chassis_link, child rotacastor_left_link, origin xyz=0.177 -0.274 0.043 rpy=0 0 0, axis 1 0 0
- added joint rotacastor_right_joint: type continuous, parent chassis_link, child rotacastor_right_link, origin xyz=-0.177 -0.274 0.043 rpy=0 0 0, axis 1 0 0
- added joint wheel_left_joint: type continuous, parent chassis_link, child wheel_left_link, origin xyz=0.247 0.157 0.058 rpy=0 0 0, axis 1 0 0, limit effort=10000 velocity=1000
- added joint wheel_right_joint: type continuous, parent chassis_link, child wheel_right_link, origin xyz=-0.247 0.157 0.058 rpy=0 0 0, axis 1 0 0, limit effort=10000 velocity=1000
